File: thelio-pwrbtn-female.kicad_pcb (KiCad board)
At the start: 2 copper layers, 14.5 x 15 mm, 0 parts

Commit message: Finish boards
Parts:
- added J1: female_blade, pwrbtn:female_blade, F.Cu at (39.2, 42.5)
- added J2: PinHeader_1x04_P2.54mm_Vertical, Connector_PinHeader_2.54mm:PinHeader_1x04_P2.54mm_Vertical, B.Cu at (35.5, 37.0)
Routing:
- net (no net): track 0.00 -> 22.1 mm
Other:
- outline, holes or cut-outs redrawn
