File: thelio-pwrbtn-female.kicad_pcb (KiCad board)
At the start: 2 copper layers, 14.5 x 15 mm, 2 parts, among them J1 female_blade, J2 PinHeader_1x04_P2.54mm_Vertic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

Commit message: Update step models
Changed lines of the file:
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@@
       (effects (font (size 1 1) (thickness 0.15)))
     )
+    (fp_line (start 7.125 4.4) (end 7.125 -1.12) (layer F.SilkS) (width 0.12))
+    (fp_line (start -7.125 4.4) (end 7.125 4.4) (layer F.SilkS) (width 0.12))
+    (fp_line (start -7.125 -1.12) (end 7.125 -1.12) (layer F.SilkS) (width 0.12))
+    (fp_line (start -7.125 4.4) (end -7.125 -1.12) (layer F.SilkS) (width 0.12))
     (fp_text user %R (at 0 -4 180) (layer F.Fab)
       (effects (font (size 1 1) (thickness 0.15)))
     )
-    (fp_line (start -7 4.5) (end -7 -1.5) (layer F.SilkS) (width 0.12))
-    (fp_line (start -7 -1.5) (end 7 -1.5) (layer F.SilkS) (width 0.12))
-    (fp_line (start -7 4.5) (end 7 4.5) (layer F.SilkS) (width 0.12))
-    (fp_line (start 7 4.5) (end 7 -1.5) (layer F.SilkS) (width 0.12))
+    (pad "" np_thru_hole circle (at -5.25 1.98 90) (size 1 1) (drill 1) (layers *.Cu *.Mask))
+    (pad "" np_thru_hole circle (at 5.25 1.98 90) (size 1 1) (drill 1) (layers *.Cu *.Mask))
+    (pad 1 thru_hole rect (at -3.75 0 90) (size 1.7 1.7) (drill 1) (layers *.Cu *.Mask))
+    (pad 2 thru_hole circle (at -1.25 0 90) (size 1.7 1.7) (drill 1) (layers *.Cu *.Mask))
+    (pad 3 thru_hole circle (at 1.25 0 90) (size 1.7 1.7) (drill 1) (layers *.Cu *.Mask))
     (pad 4 thru_hole circle (at 3.75 0 90) (size 1.7 1.7) (drill 1) (layers *.Cu *.Mask))
-    (pad 3 thru_hole circle (at 1.25 0 90) (size 1.7 1.7) (drill 1) (layers *.Cu *.Mask))
-    (pad 2 thru_hole circle (at -1.25 0 90) (size 1.7 1.7) (drill 1) (layers *.Cu *.Mask))
-    (pad 1 thru_hole rect (at -3.75 0 90) (size 1.7 1.7) (drill 1) (layers *.Cu *.Mask))
-    (pad "" np_thru_hole circle (at 5.25 1.98 90) (size 1 1) (drill 1) (layers *.Cu *.Mask))
-    (pad "" np_thru_hole circle (at -5.25 1.98 90) (size 1 1) (drill 1) (layers *.Cu *.Mask))
     (model ${KIPRJMOD}/female_blade.step
-      (offset (xyz -5.9 0.6 0))
+      (offset (xyz -5.5 1 0))
       (scale (xyz 1 1 1))
       (rotate (xyz -90 0 0))
