File: thelio-pwrbtn-male.kicad_pcb (KiCad board)
At the start: 2 copper layers, 12.5 x 15 mm, 0 parts

Commit message: Finish boards
Parts:
- added REF**: male_blade, pwrbtn:male_blade, F.Cu at (38.0, 34.0)
- added REF**: PinHeader_1x04_P2.54mm_Horizontal, Connector_PinHeader_2.54mm:PinHeader_1x04_P2.54mm_Horizontal, B.Cu at (41.8, 39.5)
Routing:
- net (no net): track 0.00 -> 23.5 mm
Other:
- outline, holes or cut-outs redrawn

Commit message: Update step models
Parts:
- renumbered REF** to J1, REF** to J2
Changed lines of the file:
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@@
     (46 B.CrtYd user)
     (47 F.CrtYd user)
-    (48 B.Fab user)
-    (49 F.Fab user)
+    (48 B.Fab user hide)
+    (49 F.Fab user hide)
   )
   (setup
@@
     (solder_mask_min_width 0.25)
     (aux_axis_origin 31.75 32)
-    (grid_origin 41.75 39.5)
+    (grid_origin 34.13 39.5)
     (visible_elements FFFFFF7F)
     (pcbplotparams
@@
     (descr "Through hole straight pin header, 1x04, 2.54mm pitch, single row")
     (tags "Through hole pin header THT 1x04 2.54mm single row")
-    (fp_text reference REF** (at 0 6) (layer F.SilkS)
+    (fp_text reference J1 (at -3.75 -2.96) (layer F.SilkS)
       (effects (font (size 1 1) (thickness 0.15)))
     )
@@
       (effects (font (size 1 1) (thickness 0.15)))
     )
+    (fp_line (start 6 2) (end 6 -2) (layer F.SilkS) (width 0.12))
+    (fp_line (start -6 -2) (end 6 -2) (layer F.SilkS) (width 0.12))
+    (fp_line (start -6 2) (end 6 2) (layer F.SilkS) (width 0.12))
+    (fp_line (start -6 2) (end -6 -2) (layer F.SilkS) (width 0.12))
     (fp_text user %R (at 0 -4) (layer F.Fab)
       (effects (font (size 1 1) (thickness 0.15)))
     )
-    (fp_line (start -6 2) (end -6 -2) (layer F.SilkS) (width 0.12))
-    (fp_line (start -6 2) (end 6 2) (layer F.SilkS) (width 0.12))
-    (fp_line (start -6 -2) (end 6 -2) (layer F.SilkS) (width 0.12))
-    (fp_line (start 6 2) (end 6 -2) (layer F.SilkS) (width 0.12))
+    (pad 1 thru_hole rect (at -3.75 0 270) (size 1.7 1.7) (drill 1) (layers *.Cu *.Mask))
+    (pad 2 thru_hole circle (at -1.25 0 270) (size 1.7 1.7) (drill 1) (layers *.Cu *.Mask))
+    (pad 3 thru_hole circle (at 1.25 0 270) (size 1.7 1.7) (drill 1) (layers *.Cu *.Mask))
     (pad 4 thru_hole circle (at 3.75 0 270) (size 1.7 1.7) (drill 1) (layers *.Cu *.Mask))
-    (pad 3 thru_hole circle (at 1.25 0 270) (size 1.7 1.7) (drill 1) (layers *.Cu *.Mask))
-    (pad 2 thru_hole circle (at -1.25 0 270) (size 1.7 1.7) (drill 1) (layers *.Cu *.Mask))
-    (pad 1 thru_hole rect (at -3.75 0 270) (size 1.7 1.7) (drill 1) (layers *.Cu *.Mask))
     (model ${KIPRJMOD}/male_blade.step
-      (offset (xyz -6.1 -1.4 0))
+      (offset (xyz -6.15 -1.5 0))
       (scale (xyz 1 1 1))
       (rotate (xyz -90 0 0))
@@
     (descr "Through hole angled pin header, 1x04, 2.54mm pitch, 6mm pin length, single row")
     (tags "Through hole angled pin header THT 1x04 2.54mm single row")
-    (fp_text reference REF** (at 4.385 2.27 90) (layer B.SilkS)
+    (fp_text reference J2 (at -2.72 0 180) (layer B.SilkS)
       (effects (font (size 1 1) (thickness 0.15)) (justify mirror))
     )
